Commit message: sia20: improve mesh quality.
This change adds:

 - detailed meshes based on CAD model offered on motoman.co.uk web site
 - updated collision meshes based on the detailed meshes

Also minor fixes to the way materials / mesh colours are configured for
the links in the collision model (must be set on the 'visual' geometry
elements, but colours are only applied to the 'collision' geometry).

No changes to the kinematic chain itself.

Thanks to @ted-miller from Motoman for providing an updated CAD model
of the SIA20.

File: motoman_sia_support/urdf/sia20_macro.xacro (robot description, xacro)
@@ -4,6 +4,24 @@
     <link name="${prefix}base_link">
       <visual>
+        <origin rpy="0 0 0" xyz="0 0 0"/>
         <geometry>
-          <mesh filename="package://motoman_sia_support/meshes/sia20/visual/base_link.stl" />
+          <mesh filename="package://motoman_sia_support/meshes/sia20/visual/base_link.dae" />
+        </geometry>
+        <material name="white">
+          <color rgba="1 1 1 1"/>
+        </material>
+      </visual>
+      <collision>
+        <origin rpy="0 0 0" xyz="0 0 0"/>
+        <geometry>
+          <mesh filename="package://motoman_sia_support/meshes/sia20/collision/base_link.stl" />
+        </geometry>
+      </collision>
+    </link>
+    <link name="${prefix}link_s">
+      <visual>
+        <origin rpy="0 0 0" xyz="0 0 0"/>
+        <geometry>
+          <mesh filename="package://motoman_sia_support/meshes/sia20/visual/link_s.dae"/>
         </geometry>
         <material name="blue">
@@ -12,44 +30,23 @@
       </visual>
       <collision>
-        <geometry>
-          <mesh filename="package://motoman_sia_support/meshes/sia20/collision/base_link.stl" />
-        </geometry>
-        <material name="yellow">
-          <color rgba="0 1 1 1"/>
-        </material>
-      </collision>
-    </link>
-    <link name="${prefix}link_s">
-      <visual>
-        <origin rpy="0 0 3.1416" xyz="0 0 0"/>
-        <geometry>
-          <mesh filename="package://motoman_sia_support/meshes/sia20/visual/link_s.stl"/>
-        </geometry>
-        <material name="silver">
-          <color rgba="0.8 0.8 0.8 1"/>
-        </material>
-      </visual>
-      <collision>
-        <origin rpy="0 0 3.1416" xyz="0 0 0"/>
+        <origin rpy="0 0 0" xyz="0 0 0"/>
         <geometry>
           <mesh filename="package://motoman_sia_support/meshes/sia20/collision/link_s.stl" />
         </geometry>
-        <material name="yellow"/>
       </collision>
     </link>
     <link name="${prefix}link_l">
       <visual>
-        <origin rpy="1.57 3.1416 3.1416" xyz="0 0 0"/>
+        <origin rpy="0 0 0" xyz="0 0 0"/>
         <geometry>
-          <mesh filename="package://motoman_sia_support/meshes/sia20/visual/link_l.stl"/>
+          <mesh filename="package://motoman_sia_support/meshes/sia20/visual/link_l.dae"/>
         </geometry>
-        <material name="blue"/>
+        <material name="white"/>
       </visual>
       <collision>
-        <origin rpy="1.57 3.1416 3.1416" xyz="0 0 0"/>
+        <origin rpy="0 0 0" xyz="0 0 0"/>
         <geometry>
           <mesh filename="package://motoman_sia_support/meshes/sia20/collision/link_l.stl"/>
         </geometry>
-        <material name="yellow"/>
       </collision>
     </link>
@@ -58,7 +55,7 @@
         <origin rpy="0 0 0" xyz="0 0 0"/>
         <geometry>
-          <mesh filename="package://motoman_sia_support/meshes/sia20/visual/link_e.stl"/>
+          <mesh filename="package://motoman_sia_support/meshes/sia20/visual/link_e.dae"/>
         </geometry>
-        <material name="silver"/>
+        <material name="white"/>
       </visual>
       <collision>
@@ -67,21 +64,19 @@
           <mesh filename="package://motoman_sia_support/meshes/sia20/collision/link_e.stl"/>
         </geometry>
-        <material name="yellow"/>
       </collision>
     </link>
     <link name="${prefix}link_u">
       <visual>
-        <origin rpy="1.57 -3.1415 3.1416" xyz="0 0 0"/>
+        <origin rpy="0 0 0" xyz="0 0 0"/>
         <geometry>
-          <mesh filename="package://motoman_sia_support/meshes/sia20/visual/link_u.stl"/>
+          <mesh filename="package://motoman_sia_support/meshes/sia20/visual/link_u.dae"/>
         </geometry>
         <material name="blue"/>
       </visual>
       <collision>
-        <origin rpy="1.57 -3.1415 3.1416" xyz="0 0 0"/>
+        <origin rpy="0 0 0" xyz="0 0 0"/>
         <geometry>
           <mesh filename="package://motoman_sia_support/meshes/sia20/collision/link_u.stl"/>
         </geometry>
-        <material name="yellow"/>
       </collision>
     </link>
@@ -90,7 +85,7 @@
         <origin rpy="0 0 0" xyz="0 0 0"/>
         <geometry>
-          <mesh filename="package://motoman_sia_support/meshes/sia20/visual/link_r.stl"/>
+          <mesh filename="package://motoman_sia_support/meshes/sia20/visual/link_r.dae"/>
         </geometry>
-        <material name="silver"/>
+        <material name="white"/>
       </visual>
       <collision>
@@ -99,35 +94,36 @@
           <mesh filename="package://motoman_sia_support/meshes/sia20/collision/link_r.stl"/>
         </geometry>
-        <material name="yellow"/>
       </collision>
     </link>
     <link name="${prefix}link_b">
       <visual>
-        <origin rpy="-1.57 0 0" xyz="0 0 0"/>
+        <origin rpy="0 0 0" xyz="0 0 0"/>
         <geometry>
-          <mesh filename="package://motoman_sia_support/meshes/sia20/visual/link_b.stl"/>
+          <mesh filename="package://motoman_sia_support/meshes/sia20/visual/link_b.dae"/>
         </geometry>
         <material name="blue"/>
       </visual>
       <collision>
-        <origin rpy="-1.57 0 0" xyz="0 0 0"/>
+        <origin rpy="0 0 0" xyz="0 0 0"/>
         <geometry>
           <mesh filename="package://motoman_sia_support/meshes/sia20/collision/link_b.stl"/>
         </geometry>
-        <material name="yellow"/>
       </collision>
     </link>
     <link name="${prefix}link_t">
       <visual>
+        <origin rpy="0 0 0" xyz="0 0 0"/>
         <geometry>
-          <mesh filename="package://motoman_sia_support/meshes/sia20/visual/link_t.stl" />
+          <mesh filename="package://motoman_sia_support/meshes/sia20/visual/link_t.dae" />
         </geometry>
-        <material name="silver"/>
+        <material name="silver">
+          <color rgba="0.45 0.45 0.45 1"/>
+        </material>
       </visual>
       <collision>
+        <origin rpy="0 0 0" xyz="0 0 0"/>
         <geometry>
           <mesh filename="package://motoman_sia_support/meshes/sia20/collision/link_t.stl" />
         </geometry>
-        <material name="yellow"/>
       </collision>
     </link>

Commit message: sia20: remove fictitious effort limits.

File: motoman_sia_support/urdf/sia20_macro.xacro (robot description, xacro)
@@ -134,5 +134,5 @@
       <origin xyz="0 0 0.41" rpy="0 0 0"/>
       <axis xyz="0 0 1" />
-      <limit lower="-3.1416" upper="3.1416" effort="100" velocity="2.26" />
+      <limit lower="-3.1416" upper="3.1416" effort="0" velocity="2.26" />
     </joint>
     <joint name="${prefix}joint_l" type="revolute">
@@ -141,5 +141,5 @@
       <origin xyz="0 0 0" rpy="0 0 0"/>
       <axis xyz="0 1 0" />
-      <limit lower="-1.91" upper="1.91" effort="100" velocity="2.26" />
+      <limit lower="-1.91" upper="1.91" effort="0" velocity="2.26" />
     </joint>
     <joint name="${prefix}joint_e" type="revolute">
@@ -148,5 +148,5 @@
       <origin xyz="0 0 0.49" rpy="0 0 0"/>
       <axis xyz="0 0 1" />
-      <limit lower="-2.96" upper="2.96" effort="100" velocity="2.96" />
+      <limit lower="-2.96" upper="2.96" effort="0" velocity="2.96" />
     </joint>
     <joint name="${prefix}joint_u" type="revolute">
@@ -155,5 +155,5 @@
       <origin xyz="0 0 0" rpy="0 0 0"/>
       <axis xyz="0 -1 0" />
-      <limit lower="-2.26" upper="2.26" effort="100" velocity="2.96" />
+      <limit lower="-2.26" upper="2.26" effort="0" velocity="2.96" />
     </joint>
     <joint name="${prefix}joint_r" type="revolute">
@@ -162,5 +162,5 @@
       <origin xyz="0 0 0.420" rpy="0 0 0"/>
       <axis xyz="0 0 -1" />
-      <limit lower="-3.1416" upper="3.1416" effort="100" velocity="3.48" />
+      <limit lower="-3.1416" upper="3.1416" effort="0" velocity="3.48" />
     </joint>
     <joint name="${prefix}joint_b" type="revolute">
@@ -169,5 +169,5 @@
       <origin xyz="0 0 0" rpy="0 0 0"/>
       <axis xyz="0 -1 0" />
-      <limit lower="-1.91" upper="1.91" effort="100" velocity="3.48" />
+      <limit lower="-1.91" upper="1.91" effort="0" velocity="3.48" />
     </joint>
     <joint name="${prefix}joint_t" type="revolute">
@@ -176,5 +176,5 @@
       <origin xyz="0 0 0.18" rpy="0 0 0"/>
       <axis xyz="0 0 -1" />
-      <limit lower="-3.1416" upper="3.1416" effort="100" velocity="6.97" />
+      <limit lower="-3.1416" upper="3.1416" effort="0" velocity="6.97" />
     </joint>
     <joint name="${prefix}link_t-tool0" type="fixed" >
